File: rev.1.0.0/BUDDY_v1.0.0.kicad_pcb (KiCad board)
At the start: 6 copper layers, 105 x 70 mm, 364 parts, among them J1 Conn_01x03, J1-jumper1 2,54 jumper, J10 Conn_02x04_Odd_Even, J11 UFL coaxial, J12 Conn_01x01, J13 Conn_01x01, J14 Conn_01x01, J15 Conn_01x01, J16 Conn_01x01, J17 Conn_01x01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

Commit message: update to new kicad
Other:
- net class Default removed
